File: HW/Kirby_SAO/Kirby_SAO.kicad_pcb (KiCad board)
At the start: 2 copper layers, 45.9 x 43.9 mm, 19 parts, among them X1 Badgelife_sao_connector_v169b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

Commit message: finial
Parts:
- removed D10, D8, D9: LED, Kirby_SAO:1204_SIDE_VIEW_LED
- added R3: 50R, Resistor_SMD:R_0805_2012Metric_Pad1.15x1.40mm_HandSolder, B.Cu at (108.5, 104.8)
- moved D6 29.2 mm to (90.5, 112.1), turned to 315 degrees
- moved D4 29.0 mm to (117.2, 99.7), turned to 180 degrees
- moved D5 19.3 mm to (114.5, 104.7), turned to 90 degrees
- moved D3 18.2 mm to (101.2, 116.0), turned to 0 degrees
- moved R2 13.7 mm to (101.7, 113.0)
- moved D7 9.07 mm to (111.5, 112.1)
- moved D2 7.63 mm to (89.8, 105.0), turned to 270 degrees
- moved R1 5.83 mm to (92.0, 100.0)
Connections:
- D3 pad 2: Net-(D1-Pad2) -> Net-(D3-Pad2)
- D4 pad 2: Net-(D1-Pad2) -> Net-(D4-Pad2)
- D5 pad 2: Net-(D1-Pad2) -> Net-(D4-Pad2)
- D6 pad 2: Net-(D10-Pad2) -> Net-(D3-Pad2)
- D7 pad 2: Net-(D10-Pad2) -> Net-(D3-Pad2)
- R2 pad 2: Net-(D10-Pad2) -> Net-(D3-Pad2)
- X1 pad 3: Net-(X1-Pad3) -> (no net)
- X1 pad 4: Net-(X1-Pad4) -> (no net)
- X1 pad 5: Net-(X1-Pad5) -> (no net)
- X1 pad 6: Net-(X1-Pad6) -> (no net)
Routing:
- net Net-(D10-Pad2): track 44.4 -> 0.00 mm
- net Net-(D1-Pad2): track 57.2 -> 16.1 mm
- net Net-(D3-Pad2): track 0.00 -> 26.1 mm
- net Net-(D4-Pad2): track 0.00 -> 10.9 mm
- net VCC: track 23.5 -> 29.1 mm
